File: Board/v1/MusicFilter.kicad_sch (KiCad schematic)
At the start: 50 parts, among them J1 TYPE-C-31-M-17, J2 FPC 0.5mm 10P, J3 Conn_01x08_Male, J4 Conn_01x02_Male, P1 SWDPins, SW1 SW_Push, SW2 SW_Push, U1 MP2359, U2 STM32F103CBUx, Y1 8MHz

Commit message: board v2 is out
Parts:
- removed C1: 10n, Capacitor_SMD:C_0603_1608Metric_Pad1.08x0.95mm_HandSolder, symbol Device:C_Small
- removed C17: 100n, Capacitor_SMD:C_0603_1608Metric_Pad1.08x0.95mm_HandSolder, symbol Device:C_Small
- removed C4: 10u, Capacitor_SMD:C_0603_1608Metric_Pad1.08x0.95mm_HandSolder, symbol Device:C_Small
- removed D1: B5819W, Diode_SMD:D_SOD-123, symbol Device:D_Schottky_Small
- removed D4: BLUE, LED_SMD:LED_0805_2012Metric_Pad1.15x1.40mm_HandSolder, symbol Device:LED_Small
- removed FB1: 600 @ 100 MHz, Inductor_SMD:L_0603_1608Metric_Pad1.05x0.95mm_HandSolder, symbol Device:FerriteBead_Small
- removed J3: Conn_01x08_Male, Connector_PinHeader_2.54mm:PinHeader_1x08_P2.54mm_Vertical, symbol Connector:Conn_01x08_Male
- removed J4: Conn_01x02_Male, Connector_PinHeader_2.54mm:PinHeader_1x02_P2.54mm_Vertical, symbol Connector:Conn_01x02_Male
- removed L1: 47u, Inductor_SMD:L_Abracon_ASPI-0630LR, symbol Device:L_Small
- removed R1: 47k, Resistor_SMD:R_0603_1608Metric_Pad0.98x0.95mm_HandSolder, symbol Device:R_Small
- removed R5: 1k5, Resistor_SMD:R_0603_1608Metric_Pad0.98x0.95mm_HandSolder, symbol Device:R_Small
- removed R9: 1k, Resistor_SMD:R_0603_1608Metric_Pad0.98x0.95mm_HandSolder, symbol Device:R_Small
- removed U1: MP2359, Package_TO_SOT_SMD:SOT-23-6_Handsoldering, symbol dannySymLib:MP2359
- removed U2: STM32F103CBUx, Package_DFN_QFN:QFN-48-1EP_7x7mm_P0.5mm_EP5.6x5.6mm, symbol MCU_ST_STM32F1:STM32F103CBUx
- removed Y1: 8MHz, Crystal:Crystal_SMD_3225-4Pin_3.2x2.5mm_HandSoldering, symbol Device:Crystal_GND24_Small
- added BT1: BK-912, DannyFootprintLibs:BK-912, symbol Device:Battery_Cell
- added C14, C20, C5: 100n, Capacitor_SMD:C_0603_1608Metric_Pad1.08x0.95mm_HandSolder, symbol Device:C_Small
- added C15, C16: 1u, Capacitor_SMD:C_0603_1608Metric_Pad1.08x0.95mm_HandSolder, symbol Device:C_Small
- added C6: 4u7, Capacitor_SMD:C_0603_1608Metric_Pad1.08x0.95mm_HandSolder, symbol Device:C_Small
- added D1, D4, D5, D6: WHITE, LED_SMD:LED_0805_2012Metric_Pad1.15x1.40mm_HandSolder, symbol Device:LED
- added IC1: TP4056X, DannyFootprintLibs:ESOP-8_L4.9-W3.9-P1.27-LS6.0-BL-EP, symbol dannySymLib:TP4056X
- added R10, R11, R12, R13: 1k5, Resistor_SMD:R_0603_1608Metric_Pad0.98x0.95mm_HandSolder, symbol Device:R_Small
- added R7: 10k, Resistor_SMD:R_0603_1608Metric_Pad0.98x0.95mm_HandSolder, symbol Device:R_Small
- added SW3, SW4: SW_Push, DannyFootprintLibs:SW_Kailh_Choc_V1_HOTSWAP, symbol Switch:SW_Push
- added SW5: SW_SPDT, Button_Switch_SMD:SW_SPDT_PCM12, symbol Switch:SW_SPDT
- added U1: STM32F401RCTx, Package_QFP:LQFP-64_10x10mm_P0.5mm, symbol MCU_ST_STM32F4:STM32F401RCTx
- added U2: LP5907MFX-3.3, Package_TO_SOT_SMD:SOT-23-5, symbol Regulator_Linear:LP5907MFX-3.3
- added Y1: 8MHz 20pF, Crystal:Crystal_SMD_5032-2Pin_5.0x3.2mm_HandSoldering, symbol Device:Crystal_Small
- C1: renamed from C15; value 12p -> 22p
- C7: renamed from C16; value 12p -> 22p
- C8: renamed from C11; value 10n -> 100n
- D3: value RED -> WHITE
- F1: value 500mA -> 200mA; footprint Fuse:Fuse_0805_2012Metric_Pad1.15x1.40mm_HandSolder -> Fuse:Fuse_0603_1608Metric_Pad1.05x0.95mm_HandSolder
- H1, H2, H3, H4: value MountingHole_Pad -> MH; footprint MountingHole:MountingHole_4.3mm_M4_Pad_Via -> MountingHole:MountingHole_2.2mm_M2_Pad_Via
- J1: renamed from J2; footprint DannyFootprintLibs:FPC 0.5mm 10P -> DannyFootprintLibs:96x96 Sharp Memory Lcd With FPC Connector 10p 0.5mm
- R2: value 15k -> 1k5
- R3: value 270 -> 17k4
- SW1, SW2: footprint DannyFootprintLibs:SW_Kailh_Choc_V1 -> DannyFootprintLibs:SW_Kailh_Choc_V1_HOTSWAP
- renumbered C6 to C10, C7 to C11, C8 to C12, C9 to C13, C13 to C17, C14 to C18, C12 to C19, C10 to C4, C5 to C9, FB2 to FB1, J1 to J2, R8 to R1, R10 to R4, R11 to R5, R4 to R8, R7 to R9
Connections:
- net BUCK_EN is gone; now on net +5V: C2.1
- net BUCK_FB is gone; now on net +5V: R2.2
- net +3.3VA: now also C20.1, U1.13 (VREF+)
- net +3V3: now also R9.2, C14.1, C16.1, R10.2, R11.2, R12.2, R13.2, SW3.2, SW4.2, U1.1 (VBAT), U1.19 (VDD), U1.32 (VDD), U1.48 (VDD), U1.64 (VDD), U2.5 (OUT); no longer C3.2, D3.2 (A)
- net +5V: now also IC1.4 (VCC), IC1.8 (CE)
- net BOOT0: now also U1.60 (BOOT0)
- net CS: now also U1.20 (PA4)
- net DISP: now also U1.22 (PA6)
- net EXTCOMM: now also U1.41 (PA8); no longer R6.1
- net GND: now also BT1.2 (-), C14.2, C15.2, C16.2, C20.2, C5.2, C6.2, IC1.1 (TEMP), IC1.3 (GND), IC1.6 (~{STDBY}), IC1.9 (EAD), R7.1, U1.12 (VSSA), U1.18 (VSS), U1.31 (VSS), U1.47 (VSS), U1.63 (VSS), U2.2 (GND); no longer R9.2
- net KEY1: now also U1.8 (PC0)
- net KEY2: now also U1.9 (PC1)
- net NRST: now also C5.1, U1.7 (NRST)
- net OSC_IN: now also U1.5 (PH0), Y1.1
- net OSC_OUT: now also U1.6 (PH1), Y1.2
- net SPI1_CLK: now also U1.21 (PA5)
- net SPI1_MOSI: now also U1.23 (PA7)
- net SWCLK: now also U1.49 (PA14)
- net SWDIO: now also U1.46 (PA13)
- net KEY1_LED: now reaches D3.1 (K)
- net KEY1_LED: now also U1.37 (PC6)
- net LDO_IN: now reaches F1.1
- net LDO_IN: now also SW5.1 (A)
- net at F1.2: now also C15.1, U2.1 (IN), U2.3 (EN)
- net at R2.1: now also D1.2 (A); no longer R3.2
- new net: D5.2 (A), R12.1
- new net: D6.2 (A), R13.1
- new net: D4.2 (A), R11.1
- new net: D3.2 (A), R10.1
- new net BAT: BT1.1 (+), C3.2, IC1.5 (BAT), SW5.2 (B)
- new net CHRG: D1.1 (K), IC1.7 (~{CHRG})
- new net KEY2_LED: D4.1 (K), U1.38 (PC7)
- new net KEY3: R6.1, SW3.1, U1.10 (PC2)
- new net KEY3_LED: D5.1 (K), U1.39 (PC8)
- new net KEY4: R7.2, SW4.1, U1.11 (PC3)
- new net KEY4_LED: D6.1 (K), U1.40 (PC9)
- new net PROG: IC1.2 (PROG), R3.2
- new net VCAP1: C6.1, U1.30 (VCAP1)
- no-connect marks 28 -> 42
Other:
- company: DannyHallo_2022 -> 2022DannyHallo
- title: MusicFilter -> Entertainment Kit
- moved on the sheet: C10, C11, C12, C13, C17, C18, C19, C2, C4, C8, C9, D2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
